File: Analog_Sandbox_PCB/Analog_Sandbox_PCB.kicad_pcb (KiCad board)
At the start: 2 copper layers, 203.2 x 101.6 mm, 105 parts, among them J1 PAD, J10 PAD, J13 PAD, J14 PAD, J15 PAD, J16 PAD, J19 PAD, J2 PAD, J20 PAD, J23 PAD, J25 PAD, J27 PAD, J28 PAD, J29 PAD, J3 PAD, J31 PAD, J32 PAD, J33 PAD, J34 PAD, J35 PAD, J36 PAD, J37 PAD, J38 PAD, J39 PAD, J41 PAD, J42 PAD, J44 PAD, J45 PAD, J46 PAD, U1 ICM7555_DIP, U2 LM358_SOIC, U3 LM334Z/LFT1

Commit message: more changes
Parts:
- added B1: ~, Battery:BatteryHolder_MYOUNG_BS-07-A1BJ001_CR2032, F.Cu at (17.4, 123.8)
- added R14: 1000, Resistor_SMD:R_2010_5025Metric_Pad1.40x2.65mm_HandSolder, F.Cu at (17.9, 140.5)
- added R15: 1000, Resistor_SMD:R_2010_5025Metric_Pad1.40x2.65mm_HandSolder, F.Cu at (17.9, 144.8)
- added R16: R, Resistor_SMD:R_2010_5025Metric_Pad1.40x2.65mm_HandSolder, F.Cu at (27.6, 140.5)
- added R17: R, Resistor_SMD:R_2010_5025Metric_Pad1.40x2.65mm_HandSolder, F.Cu at (27.6, 144.8)
- C2, C3: value (none) -> C; footprint CAPC1005X60_16997205 -> Capacitor_SMD:C_0805_2012Metric_Pad1.18x1.45mm_HandSolder
- D1, D2, D3, D4: value CHIP-FLAT-Y_0603-0.35MM -> LED; footprint LEDC1608X35N_FLAT-Y_22900745 -> Diode_SMD:D_2010_5025Metric_Pad1.52x2.65mm_HandSolder
- D5, D6, D8: value CHIP-FLAT-Y_0603-0.35MM -> ~; footprint LEDC1608X35N_FLAT-Y_22900745 -> Diode_SMD:D_2010_5025Metric_Pad1.52x2.65mm_HandSolder
- D7: value LED_CHIP_RED-1608 -> ~; footprint LEDC1608X39N_R_16378487 -> Diode_SMD:D_2010_5025Metric_Pad1.52x2.65mm_HandSolder
- J1: footprint 2.54_1.0_16378166 -> TestPoint:TestPoint_Loop_D2.50mm_Drill1.0mm
- R1: value 1000 -> R; footprint RESC1005X40_16378527 -> Resistor_SMD:R_2010_5025Metric_Pad1.40x2.65mm_HandSolder
- R10: value 1000 -> 6000; footprint RESC1005X40_16378527 -> Resistor_SMD:R_2010_5025Metric_Pad1.40x2.65mm_HandSolder
- R11: value 1000 -> 2000; footprint RESC1005X40_16378527 -> Resistor_SMD:R_2010_5025Metric_Pad1.40x2.65mm_HandSolder
- R12, R13: value (none) -> 560; footprint RESC1005X40_16378527 -> Resistor_SMD:R_2010_5025Metric_Pad1.40x2.65mm_HandSolder
- R18, R19: value (none) -> R; footprint RESC1005X40_16378527 -> Resistor_SMD:R_2010_5025Metric_Pad1.40x2.65mm_HandSolder
- R2: value 2000 -> R; footprint RESC1005X40_16378527 -> Resistor_SMD:R_2010_5025Metric_Pad1.40x2.65mm_HandSolder
- R3: value 1000 -> 560; footprint RESC1005X40_16378527 -> Resistor_SMD:R_2010_5025Metric_Pad1.40x2.65mm_HandSolder
- R4: value 2000 -> 560; footprint RESC1005X40_16378527 -> Resistor_SMD:R_2010_5025Metric_Pad1.40x2.65mm_HandSolder
- R5: value 560 -> 1000; footprint RESC1005X40_16378527 -> Resistor_SMD:R_2010_5025Metric_Pad1.40x2.65mm_HandSolder
- R6: value 560 -> 2000; footprint RESC1005X40_16378527 -> Resistor_SMD:R_2010_5025Metric_Pad1.40x2.65mm_HandSolder
- R7: value 3000 -> 1000; footprint RESC1005X40_16378527 -> Resistor_SMD:R_2010_5025Metric_Pad1.40x2.65mm_HandSolder
- R8: footprint RESC1005X40_16378527 -> Resistor_SMD:R_2010_5025Metric_Pad1.40x2.65mm_HandSolder
- R9: value 6000 -> 3000; footprint RESC1005X40_16378527 -> Resistor_SMD:R_2010_5025Metric_Pad1.40x2.65mm_HandSolder
- S10: value DS01E -> ~
- S3, S4, S5, S6, S7, S8, S9: value DS01E -> SWITCH
- U1: value ICM7555_DIP -> Current Source
- VR1: value 3362P-1-102LF -> <OUTPUT VOLTAGE>
- VR2, VR3, VR4, VR5, VR6: value 3362P-1-102LF -> ~
Connections:
- C2 pad 1: N$49 -> V_Reg_Out
- C2 pad 2: N$52 -> GND
- C3 pad 1: N$52 -> /Vin
- C3 pad 2: N$48 -> GND
- D7 pad 1: N$47 -> (no net)
- D7 pad 2: N$18 -> (no net)
- J1 pad 1: N$2 -> Net-(J1-P)
- J10 pad 1: N$7 -> GND
- J13 pad 1: N$15 -> Net-(J13-P)
- J14 pad 1: N$10 -> Net-(J14-P)
- J15 pad 1: N$11 -> Net-(J15-P)
- J16 pad 1: N$52 -> Net-(J16-P)
- J2 pad 1: N$52 -> Net-(J2-P)
- J3 pad 1: N$52 -> Net-(J3-P)
- R1 pad 1: N$2 -> V_Reg_Out
- R1 pad 2: N$7 -> Net-(VR1-ADJ)
- R10 pad 1: N$8 -> Net-(R10-Pad1)
- R10 pad 2: N$16 -> GND
- R11 pad 1: N$17 -> Net-(R11-Pad1)
- R11 pad 2: N$16 -> GND
- R12 pad 1: N$52 -> Net-(R12-Pad1)
- R12 pad 2: N$29 -> Net-(D3-PadA)
- R13 pad 1: N$53 -> Net-(J8-P)
- R13 pad 2: N$36 -> Net-(D4-PadA)
- R18 pad 1: N$34 -> Net-(VR5-CW)
- R18 pad 2: N$1 -> Net-(J14-P)
- R19 pad 1: N$20 -> Net-(VR6-CW)
- R19 pad 2: N$21 -> Net-(J15-P)
- R2 pad 1: N$7 -> GND
- R2 pad 2: N$52 -> Net-(VR1-ADJ)
- R3 pad 1: N$15 -> Net-(J1-P)
- R3 pad 2: N$10 -> Net-(D1-PadA)
- R4 pad 1: N$10 -> Net-(R4-Pad1)
- R4 pad 2: N$11 -> Net-(D2-PadA)
- R5 pad 1: N$2 -> Net-(R4-Pad1)
- R5 pad 2: N$4 -> Net-(J2-P)
- R6 pad 1: N$2 -> Net-(J3-P)
- R6 pad 2: N$5 -> unconnected-(R6-Pad2)
- R7 pad 1: N$11 -> Net-(J4-P)
- R7 pad 2: N$52 -> Net-(J5-P)
- R8 pad 1: N$12 -> Net-(J5-P)
- R8 pad 2: N$52 -> Net-(J6-P)
- R9 pad 1: N$14 -> Net-(J6-P)
- R9 pad 2: N$52 -> GND
- S10 pad 1: N$36 -> V_Reg_Out
- S10 pad 2: N$34 -> unconnected-(S10-Pad2)
- S3 pad 1: N$36 -> unconnected-(S3-Pad1)
- S3 pad 2: N$2 -> Net-(R11-Pad1)
- S4 pad 1: N$15 -> V_Reg_Out
- S4 pad 2: N$36 -> Net-(R12-Pad1)
- S5 pad 1: N$10 -> V_Reg_Out
- S5 pad 2: N$14 -> Net-(J8-P)
- S6 pad 1: N$11 -> Net-(R15-Pad2)
- S6 pad 2: N$12 -> Net-(J11-P)
- S7 pad 1: N$36 -> unconnected-(S7-Pad1)
- S7 pad 2: N$8 -> GND
- S8 pad 1: N$17 -> V_Reg_Out
- S8 pad 2: N$9 -> Net-(J12-P)
- S9 pad 1: N$54 -> unconnected-(S9-Pad1)
- S9 pad 2: N$52 -> GND
- U1 pad 1: N$52 -> unconnected-(U1-V+-Pad1)
- U1 pad 2: N$48 -> unconnected-(U1-R-Pad2)
- U1 pad 3: N$31 -> unconnected-(U1-V--Pad3)
- U1 pad 4: N$36 -> (no net)
- U1 pad 5: N$49 -> (no net)
- U1 pad 6: N$48 -> (no net)
- U1 pad 7: N$50 -> (no net)
- U1 pad 8: N$46 -> (no net)
- VR1 pad 1: N$54 -> Net-(VR1-ADJ)
- VR1 pad 2: (no net) -> V_Reg_Out
- VR1 pad 3: N$9 -> /Vin
- VR2 pad 1: N$40 -> Net-(J11-P)
- VR2 pad 2: (no net) -> unconnected-(VR2-WIPER-Pad2)
- VR2 pad 3: N$39 -> Net-(J9-P)
- VR3 pad 1: N$45 -> Net-(VR3-CCW)
- VR3 pad 2: (no net) -> unconnected-(VR3-WIPER-Pad2)
- VR3 pad 3: N$32 -> Net-(VR3-CW)
- VR4 pad 1: N$50 -> Net-(VR4-CCW)
- VR4 pad 2: (no net) -> unconnected-(VR4-WIPER-Pad2)
- VR4 pad 3: N$48 -> Net-(VR4-CW)
- VR5 pad 1: N$19 -> Net-(VR5-CCW)
- VR5 pad 2: (no net) -> unconnected-(VR5-WIPER-Pad2)
- VR5 pad 3: N$1 -> Net-(VR5-CW)
- VR6 pad 1: N$22 -> Net-(VR6-CCW)
- VR6 pad 2: (no net) -> unconnected-(VR6-WIPER-Pad2)
- VR6 pad 3: N$21 -> Net-(VR6-CW)

Commit message: All Circuits Added, Layout Almost done
Parts:
- removed C1: , CAPC1005X60_16290819
- removed C4, C5, C6: , CAPC1005X60_16997205
- removed D10: CHIP-FLAT-Y_0603-0.35MM, LEDC1608X35N_FLAT-Y_22900745
- removed D11, D12: DIODE_DO-213AA(SOD-80), DIOMELF3516_16378169
- removed J13, J15, J19, J20, J23, J25, J27, J28, J29, J31, J32, J33, J34, J35, J36, J37, J38, J39, J41, J42, J44, J45, J46: PAD, 2.54_1.0_16378166
- removed R30, R31, R32, R34, R35: , RESC1005X40_16378527
- removed R37: 560, RESC1005X40_16378527
- removed U$1: BATTERYGENERIC, BATTERY-GENERIC_30890021
- removed U3: LM334Z/LFT1, TO92260P521H934-3_vf.hGffbZ2ORuCqFQmqaGxY-w
- removed VR1: <OUTPUT VOLTAGE>, TRIM_3362P-1-102LF_vf.A5S3VpQGRRqLSuxbPYtLvA
- removed VR4: ~, TRIM_3362P-1-102LF_vf.A5S3VpQGRRqLSuxbPYtLvA
- removed VR7, VR8: 3362P-1-102LF, TRIM_3362P-1-102LF_vf.A5S3VpQGRRqLSuxbPYtLvA
- removed VR9: LM317T, TO254P1054X470X1955-3_vf.v8R9yl4NRtKAz-4LSZOHhg
- added J17: PAD, TestPoint:TestPoint_Pad_2.5x2.5mm, F.Cu at (128.1, 72.0)
- added J4: PAD, TestPoint:TestPoint_Pad_2.5x2.5mm, F.Cu at (152.9, 98.7)
- added J5: PAD, TestPoint:TestPoint_Pad_2.5x2.5mm, F.Cu at (163.7, 88.4)
- added J6: PAD, TestPoint:TestPoint_Pad_2.5x2.5mm, F.Cu at (163.7, 78.4)
- added J7: PAD, TestPoint:TestPoint_Pad_2.5x2.5mm, F.Cu at (160.0, 69.5)
- added Q1: 2N3904, Package_TO_SOT_THT:TO-92_Inline, F.Cu at (51.6, 50.6)
- added R20: 33, Resistor_SMD:R_1206_3216Metric, F.Cu at (213.6, 87.1)
- added R21: 100, Resistor_SMD:R_1206_3216Metric, F.Cu at (69.5, 120.3)
- added R29: 1k, Resistor_SMD:R_1206_3216Metric, F.Cu at (45.7, 53.7)
- added S1: SWITCH, Button_Switch_THT:SW_DIP_SPSTx01_Slide_9.78x4.72mm_W7.62mm_P2.54mm, F.Cu at (96.0, 78.2)
- added S2: SWITCH, Button_Switch_THT:SW_DIP_SPSTx01_Slide_9.78x4.72mm_W7.62mm_P2.54mm, F.Cu at (168.9, 78.4)
- D1, D2, D3, D4: footprint Diode_SMD:D_2010_5025Metric_Pad1.52x2.65mm_HandSolder -> Diode_SMD:D_1206_3216Metric
- D5, D6, D7, D8: value ~ -> LED; footprint Diode_SMD:D_2010_5025Metric_Pad1.52x2.65mm_HandSolder -> Diode_SMD:D_1206_3216Metric
- D9: value CHIP-FLAT-Y_0603-0.35MM -> LED; footprint LEDC1608X35N_FLAT-Y_22900745 -> Diode_SMD:D_1206_3216Metric
- J1: footprint TestPoint:TestPoint_Loop_D2.50mm_Drill1.0mm -> TestPoint:TestPoint_Pad_2.5x2.5mm
- J2, J3: footprint 2.54_1.0_16378166 -> TestPoint:TestPoint_Pad_2.5x2.5mm
- R1, R10, R11, R12, R13, R14, R15, R2, R3, R4, R5, R6, R7, R8, R9: footprint Resistor_SMD:R_2010_5025Metric_Pad1.40x2.65mm_HandSolder -> Resistor_SMD:R_1206_3216Metric
- R16, R17, R18, R19: value R -> 100; footprint Resistor_SMD:R_2010_5025Metric_Pad1.40x2.65mm_HandSolder -> Resistor_SMD:R_1206_3216Metric
- R22, R23, R25, R27: value (none) -> 10k; footprint RESC1005X40_16378527 -> Resistor_SMD:R_1206_3216Metric
- R24: value (none) -> 220; footprint RESC1005X40_16378527 -> Resistor_SMD:R_1206_3216Metric
- R26: value 560 -> 10k; footprint RESC1005X40_16378527 -> Resistor_SMD:R_1206_3216Metric
- R28: value (none) -> 4.7k; footprint RESC1005X40_16378527 -> Resistor_SMD:R_1206_3216Metric
- S10: value ~ -> SWITCH; footprint DS-01_16378657 -> Button_Switch_THT:SW_DIP_SPSTx01_Slide_9.78x4.72mm_W7.62mm_P2.54mm
- S11, S12, S13, S14, S15, S16, S17, S18, S19: value DS01E -> SWITCH; footprint DS-01_16378657 -> Button_Switch_THT:SW_DIP_SPSTx01_Slide_9.78x4.72mm_W7.62mm_P2.54mm
- S3, S4, S5, S6, S7, S8, S9: footprint DS-01_16378657 -> Button_Switch_THT:SW_DIP_SPSTx01_Slide_9.78x4.72mm_W7.62mm_P2.54mm
- U1: footprint DIP826W53P254L959H508Q8B_18568598 -> Connector_PinSocket_2.54mm:PinSocket_1x03_P2.54mm_Vertical
- U2: value LM358_SOIC -> NE555P; footprint SOIC127P600X175-8N_16378340 -> Package_DIP:DIP-8_W7.62mm
- moved S16 240.9 mm to (22.6, 24.0), turned to 0 degrees
- moved S15 235.4 mm to (1.44, 36.8), turned to 0 degrees
- moved S17 231.0 mm to (22.6, 30.4), turned to 0 degrees
- moved S14 229.2 mm to (1.44, 22.0), turned to 0 degrees
- moved R15 220.8 mm to (226.7, 73.2)
- moved R14 210.8 mm to (217.6, 73.2)
- moved U2 210.6 mm to (1.08, 42.0), turned to 0 degrees
- moved S13 187.9 mm to (1.44, 15.6), turned to 0 degrees
- moved S8 178.8 mm to (57.2, 120.2), turned to 0 degrees
- moved S9 176.8 mm to (59.3, 145.7), turned to 0 degrees
- moved S12 166.3 mm to (1.44, 9.13), turned to 0 degrees
- moved R13 164.0 mm to (218.2, 66.7), turned to 0 degrees
- moved D4 163.8 mm to (227.1, 66.7), turned to 180 degrees
- moved R28 160.0 mm to (45.7, 49.5)
- moved S19 159.0 mm to (43.8, 44.2), turned to 0 degrees
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Connections:
- D1 pad 1: (no net) -> GND
- D1 pad 2: (no net) -> Net-(D1-A)
- D2 pad 1: (no net) -> Net-(D2-K)
- D2 pad 2: (no net) -> Net-(D2-A)
- D3 pad 1: (no net) -> GND
- D3 pad 2: (no net) -> Net-(D3-A)
- D4 pad 1: (no net) -> GND
- D4 pad 2: (no net) -> Net-(D4-A)
- D5 pad 1: (no net) -> Net-(D5-K)
- D5 pad 2: (no net) -> Net-(D5-A)
- D6 pad 1: (no net) -> Net-(D6-K)
- D6 pad 2: (no net) -> Net-(D6-A)
- D7 pad 1: (no net) -> Net-(D7-K)
- D7 pad 2: (no net) -> Net-(D7-A)
- D8 pad 1: (no net) -> Net-(D7-K)
- D8 pad 2: (no net) -> Net-(D8-A)
- J14 pad 1: Net-(J14-P) -> Net-(D5-K)
- J16 pad 1: Net-(J16-P) -> Net-(D7-K)
- J3 pad 1: Net-(J3-P) -> GND
- R12 pad 1: Net-(R12-Pad1) -> Net-(J7-P)
- R12 pad 2: Net-(D3-PadA) -> Net-(D3-A)
- R13 pad 2: Net-(D4-PadA) -> Net-(D4-A)
- R14 pad 2: Net-(R14-Pad2) -> Net-(U1-V+)
- R15 pad 1: Net-(R14-Pad2) -> Net-(U1-V+)
- R16 pad 2: Net-(VR3-CCW) -> Net-(VR3-CW)
- R17 pad 1: Net-(J14-P) -> Net-(D5-K)
- R18 pad 2: Net-(J14-P) -> Net-(D5-K)
- R19 pad 2: Net-(J15-P) -> Net-(D6-K)
- R22 pad 1: N$26 -> GND
- R22 pad 2: N$23 -> Net-(U2-TR)
- R23 pad 2: N$20 -> Net-(U2-R)
- R24 pad 1: N$31 -> Net-(U2-Q)
- R24 pad 2: N$13 -> Net-(D9-A)
- R25 pad 1: N$52 -> Net-(R25-Pad1)
- R25 pad 2: N$47 -> Net-(R25-Pad2)
- R26 pad 1: N$15 -> Net-(R25-Pad1)
- R26 pad 2: N$3 -> Net-(VR8-CW)
- R27 pad 1: N$35 -> Net-(R27-Pad1)
- R27 pad 2: N$32 -> Net-(R25-Pad1)
- R28 pad 1: N$52 -> Net-(Q1-B)
- R28 pad 2: N$30 -> Net-(J19-P)
- R3 pad 1: Net-(J1-P) -> Net-(J2-P)
- R3 pad 2: Net-(D1-PadA) -> Net-(D1-A)
- R4 pad 1: Net-(R4-Pad1) -> Net-(J2-P)
- R4 pad 2: Net-(D2-PadA) -> Net-(D2-A)
- R5 pad 1: Net-(R4-Pad1) -> Net-(J2-P)
- R5 pad 2: Net-(J2-P) -> Net-(J1-P)
- R6 pad 1: Net-(J3-P) -> GND
- R6 pad 2: unconnected-(R6-Pad2) -> Net-(J1-P)
- R7 pad 1: Net-(J4-P) -> Net-(J7-P)
- R8 pad 2: Net-(J6-P) (its old number) -> Net-(J5-P)
- R9 pad 1: Net-(J6-P) (its old number) -> Net-(J5-P)
- S10 pad 1: V_Reg_Out -> Net-(U2-R)
- S10 pad 2: unconnected-(S10-Pad2) -> Net-(U2-TR)
- S11 pad 1: N$52 -> Net-(J12-P)
- S11 pad 2: N$33 -> Net-(D5-K)
- S12 pad 1: N$46 -> Net-(D5-K)
- S12 pad 2: N$36 -> Net-(D6-K)
- S13 pad 1: N$36 -> Net-(D6-K)
- S13 pad 2: N$35 -> Net-(D7-K)
- S14 pad 1: N$36 -> Net-(D5-K)
- S14 pad 2: N$42 -> Net-(D7-K)
- S15 pad 1: N$52 -> V_Reg_Out
- S15 pad 2: N$41 -> Net-(U2-R)
- S16 pad 1: N$41 -> V_Reg_Out
- S16 pad 2: N$40 -> Net-(R25-Pad2)
- S17 pad 1: N$37 -> Net-(R27-Pad1)
- S18 pad 1: N$43 -> GND
- S18 pad 2: N$18 -> Net-(VR8-CW)
- S19 pad 1: N$51 -> V_Reg_Out
- S19 pad 2: N$36 -> Net-(Q1-C)
- S3 pad 1: unconnected-(S3-Pad1) -> Net-(J5-P)
- S4 pad 2: Net-(R12-Pad1) -> Net-(J7-P)
- S7 pad 1: unconnected-(S7-Pad1) -> GND
- S7 pad 2: GND -> Net-(J9-P)
- S8 pad 2: Net-(J12-P) -> Net-(R21-Pad2)
- S9 pad 1: unconnected-(S9-Pad1) -> GND
- S9 pad 2: GND -> Net-(D7-K)
- U1 pad 1: unconnected-(U1-V+-Pad1) -> Net-(U1-V+)
- U1 pad 2: unconnected-(U1-R-Pad2) -> Net-(U1-R)
- U1 pad 3: unconnected-(U1-V--Pad3) -> GND
- U2 pad 1: N$44 -> GND
- U2 pad 2: N$30 -> Net-(U2-TR)
- U2 pad 3: N$45 -> Net-(U2-Q)
- U2 pad 4: N$52 -> Net-(U2-R)
- U2 pad 5: (no net) -> Net-(U2-CV)
- U2 pad 6: (no net) -> Net-(U2-DIS)
- U2 pad 7: (no net) -> Net-(U2-DIS)
- U2 pad 8: N$51 -> Net-(U2-R)
- VR2 pad 1: Net-(J11-P) -> unconnected-(VR2-CCW-Pad1)
- VR2 pad 2: unconnected-(VR2-WIPER-Pad2) -> Net-(J11-P)
- VR3 pad 1: Net-(VR3-CCW) -> unconnected-(VR3-CCW-Pad1)
- VR3 pad 2: unconnected-(VR3-WIPER-Pad2) -> Net-(D5-A)
- VR5 pad 1: Net-(VR5-CCW) -> unconnected-(VR5-CCW-Pad1)
- VR5 pad 2: unconnected-(VR5-WIPER-Pad2) -> Net-(D7-A)
- VR6 pad 1: Net-(VR6-CCW) -> unconnected-(VR6-CCW-Pad1)
- VR6 pad 2: unconnected-(VR6-WIPER-Pad2) -> Net-(D8-A)

Commit message: fin
Parts:
- removed B1: ~, Battery:BatteryHolder_MYOUNG_BS-07-A1BJ001_CR2032
- removed C2, C3: C, Capacitor_SMD:C_0805_2012Metric_Pad1.18x1.45mm_HandSolder
- removed J16: PAD, 2.54_1.0_16378166
- removed J17: PAD, TestPoint:TestPoint_Pad_2.5x2.5mm
- removed VR2, VR3, VR5, VR6: ~, TRIM_3362P-1-102LF_vf.A5S3VpQGRRqLSuxbPYtLvA
- added BT1: Battery_Cell, Battery:BatteryHolder_Keystone_1060_1x2032, B.Cu at (61.3, 138.1)
- added BT2: Battery_Cell, Battery:BatteryHolder_Keystone_1060_1x2032, B.Cu at (61.3, 104.9)
- added Base1: PAD, TestPoint:TestPoint_Loop_D2.50mm_Drill1.85mm, F.Cu at (228.2, 129.3)
- added C1: 0.01u, Capacitor_SMD:C_1206_3216Metric, F.Cu at (183.4, 143.1)
- added C4: 47u, Capacitor_SMD:C_1206_3216Metric, F.Cu at (188.3, 143.1)
- added D10: LED, Diode_SMD:D_1206_3216Metric, F.Cu at (84.8, 135.6)
- added D11: LED, Diode_SMD:D_1206_3216Metric, F.Cu at (164.8, 139.1)
- added D12: LED, Diode_SMD:D_1206_3216Metric, F.Cu at (213.9, 141.7)
- added D13: LED, Diode_SMD:D_1206_3216Metric, F.Cu at (211.3, 86.4)
- added Emitter1: PAD, TestPoint:TestPoint_Loop_D2.50mm_Drill1.85mm, F.Cu at (236.2, 140.1)
- added J11: PAD, TestPoint:TestPoint_Loop_D2.50mm_Drill1.85mm, F.Cu at (193.7, 77.6)
- added J12: PAD, TestPoint:TestPoint_Loop_D2.50mm_Drill1.85mm, F.Cu at (92.5, 115.6)
- added J13: PAD, TestPoint:TestPoint_Loop_D2.50mm_Drill1.85mm, F.Cu at (96.2, 145.8)
- added J15: PAD, TestPoint:TestPoint_Loop_D2.50mm_Drill1.85mm, F.Cu at (144.9, 127.5)
- added J21: PAD, TestPoint:TestPoint_Loop_D2.50mm_Drill1.85mm, F.Cu at (196.8, 127.1)
- added J8: PAD, TestPoint:TestPoint_Loop_D2.50mm_Drill1.85mm, F.Cu at (166.9, 66.2)
- added J9: PAD, TestPoint:TestPoint_Loop_D2.50mm_Drill1.85mm, F.Cu at (193.2, 97.4)
- added Q2: PAD, TestPoint:TestPoint_Loop_D2.50mm_Drill1.85mm, F.Cu at (174.0, 137.8)
- added R30: 3362P-1-103LF, Sandbox:POT_3362P, F.Cu at (133.2, 120.4)
- added R31: 3362P-1-103LF, Sandbox:POT_3362P, F.Cu at (193.5, 86.7)
- added R32: 3362P-1-103LF, Sandbox:POT_3362P, F.Cu at (99.8, 120.4)
- added R33: 3362P-1-103LF, Sandbox:POT_3362P, F.Cu at (116.6, 129.7)
- added R34: 3362P-1-103LF, Sandbox:POT_3362P, F.Cu at (138.0, 145.5)
- added R35: 3362P-1-103LF, Sandbox:POT_3362P, F.Cu at (192.5, 136.8)
- added R36: 3362P-1-103LF, Sandbox:POT_3362P, F.Cu at (221.7, 131.6)
- added R37: 3362P-1-103LF, Sandbox:POT_3362P, F.Cu at (241.4, 86.4)
- added R38: 560, Resistor_SMD:R_1206_3216Metric, F.Cu at (213.9, 131.7)
- added R39: 560, Resistor_SMD:R_1206_3216Metric, F.Cu at (211.3, 79.1)
- J1, J2, J3, J4, J5, J6, J7: footprint TestPoint:TestPoint_Pad_2.5x2.5mm -> TestPoint:TestPoint_Loop_D2.50mm_Drill1.85mm
- J10, J14: footprint 2.54_1.0_16378166 -> TestPoint:TestPoint_Loop_D2.50mm_Drill1.85mm
- Q1: footprint Package_TO_SOT_THT:TO-92_Inline -> Connector_PinHeader_2.54mm:PinHeader_1x03_P2.54mm_Vertical
- R1, R2: value R -> 560
- moved R29 215.1 mm to (240.9, 143.9), turned to -90 degrees
- moved S17 211.4 mm to (230.0, 71.3)
- moved Q1 208.0 mm to (240.9, 136.7), turned to 180 degrees
- moved R28 204.0 mm to (231.3, 134.1), turned to 180 degrees
- moved R23 199.9 mm to (192.5, 124.8), turned to 90 degrees
- moved U2 196.0 mm to (177.7, 127.0)
- moved S10 194.9 mm to (171.3, 125.9), turned to -90 degrees
- moved S18 194.0 mm to (207.2, 96.7)
- moved R22 193.6 mm to (171.3, 143.1), turned to 90 degrees
- moved R27 193.5 mm to (225.3, 71.2), turned to 180 degrees
- moved D9 193.2 mm to (177.7, 145.0), turned to 90 degrees
- moved R26 192.9 mm to (220.2, 83.9), turned to -90 degrees
- moved R24 192.5 mm to (177.7, 140.3), turned to -90 degrees
- moved R25 187.5 mm to (217.0, 71.2), turned to 180 degrees
- moved S16 187.3 mm to (203.8, 71.4)
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Connections:
- J10 pad 1: GND -> Net-(D2-K)
- R1 pad 1: V_Reg_Out -> Net-(R1-Pad1)
- R1 pad 2: Net-(VR1-ADJ) -> Net-(D10-A)
- R2 pad 1: GND -> Net-(U2-R)
- R2 pad 2: Net-(VR1-ADJ) -> Net-(D11-A)
- R21 pad 2: Net-(R21-Pad2) -> Net-(R1-Pad1)
- S8 pad 2: Net-(R21-Pad2) -> Net-(R1-Pad1)
Routing:
- net GND: track 0.00 -> 122.8 mm, vias 0 -> 12
- net Net-(D7-K): track 0.00 -> 62.1 mm
- net Net-(R26-Pad2): track 0.00 -> 56.9 mm
- net Net-(U2-R): track 0.00 -> 53.7 mm
- net Net-(D5-K): track 0.00 -> 46.8 mm
- net Net-(Q1-C): track 0.00 -> 43.2 mm
- net Net-(D6-K): track 0.00 -> 43.1 mm
- net Net-(J2-P): track 0.00 -> 23.6 mm
- net Net-(J1-P): track 0.00 -> 22.5 mm
- net Net-(J8-P): track 0.00 -> 19.7 mm
- net Net-(R10-Pad1): track 0.00 -> 18.8 mm
- net Net-(J7-P): track 0.00 -> 18.7 mm
- net Net-(R25-Pad1): track 0.00 -> 16.6 mm
- net Net-(J9-P): track 0.00 -> 16.5 mm
- net Net-(U2-DIS): track 0.00 -> 16.2 mm
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- added copper zone on F.Cu, net GND
- added copper zone on B.Cu, net V_Reg_Out

Commit message: made changes from morning of 4/13
Parts:
- removed Base1, Emitter1, J1, J10, J11, J12, J13, J14, J15, J2, J21, J3, J4, J5, J6, J7, J8, J9, Q2: PAD, TestPoint:TestPoint_Loop_D2.50mm_Drill1.85mm
- removed R22: 10k, Resistor_SMD:R_1206_3216Metric
- removed S10: SWITCH, Button_Switch_THT:SW_DIP_SPSTx01_Slide_9.78x4.72mm_W7.62mm_P2.54mm
- added A1: PAD, TestPoint:TestPoint_Loop_D2.50mm_Drill1.85mm, F.Cu at (66.4, 67.4)
- added A2: PAD, TestPoint:TestPoint_Loop_D2.50mm_Drill1.85mm, F.Cu at (88.9, 73.8)
- added A3: PAD, TestPoint:TestPoint_Loop_D2.50mm_Drill1.85mm, F.Cu at (92.7, 94.1)
- added A4: PAD, TestPoint:TestPoint_Loop_D2.50mm_Drill1.85mm, F.Cu at (88.9, 67.4)
- added B1: PAD, TestPoint:TestPoint_Loop_D2.50mm_Drill1.85mm, F.Cu at (117.3, 69.5)
- added B2: PAD, TestPoint:TestPoint_Loop_D2.50mm_Drill1.85mm, F.Cu at (121.0, 78.4)
- added B3: PAD, TestPoint:TestPoint_Loop_D2.50mm_Drill1.85mm, F.Cu at (121.0, 88.4)
- added B4: PAD, TestPoint:TestPoint_Loop_D2.50mm_Drill1.85mm, F.Cu at (110.2, 98.7)
- added E1: PAD, TestPoint:TestPoint_Loop_D2.50mm_Drill1.85mm, F.Cu at (92.5, 115.6)
- added E2: PAD, TestPoint:TestPoint_Loop_D2.50mm_Drill1.85mm, F.Cu at (116.6, 119.4)
- added E3: PAD, TestPoint:TestPoint_Loop_D2.50mm_Drill1.85mm, F.Cu at (144.9, 127.5)
- added E4: PAD, TestPoint:TestPoint_Loop_D2.50mm_Drill1.85mm, F.Cu at (96.1, 145.8)
- added F1: PAD, TestPoint:TestPoint_Loop_D2.50mm_Drill1.85mm, F.Cu at (174.0, 137.8)
- added F2: PAD, TestPoint:TestPoint_Loop_D2.50mm_Drill1.85mm, F.Cu at (196.8, 127.1)
- added G1: PAD, TestPoint:TestPoint_Loop_D2.50mm_Drill1.85mm, F.Cu at (221.7, 125.0)
- added G2: PAD, TestPoint:TestPoint_Loop_D2.50mm_Drill1.85mm, F.Cu at (228.2, 129.3)
- added G3: PAD, TestPoint:TestPoint_Loop_D2.50mm_Drill1.85mm, F.Cu at (235.8, 129.3)
- added G4: PAD, TestPoint:TestPoint_Loop_D2.50mm_Drill1.85mm, F.Cu at (236.2, 140.1)
- added K1: PAD, TestPoint:TestPoint_Loop_D2.50mm_Drill1.85mm, F.Cu at (220.2, 77.0)
- added K2: PAD, TestPoint:TestPoint_Loop_D2.50mm_Drill1.85mm, F.Cu at (241.4, 75.3)
- added K3: PAD, TestPoint:TestPoint_Loop_D2.50mm_Drill1.85mm, F.Cu at (241.4, 96.6)
- added M1: PAD, TestPoint:TestPoint_Loop_D2.50mm_Drill1.85mm, F.Cu at (166.9, 66.2)
- added M2: PAD, TestPoint:TestPoint_Loop_D2.50mm_Drill1.85mm, F.Cu at (193.7, 77.6)
- added M3: PAD, TestPoint:TestPoint_Loop_D2.50mm_Drill1.85mm, F.Cu at (193.2, 97.4)
Connections:
- C4 pad 1: Net-(U2-DIS) -> Net-(C4-Pad1)
- R23 pad 1: Net-(J21-P) -> Net-(F2-P)
- R35 pad 1: GND -> Net-(C4-Pad1)
- R35 pad 2: Net-(U2-DIS) -> Net-(U2-THR)
- R35 pad 3: Net-(J21-P) -> Net-(F2-P)
- U2 pad 2: Net-(U2-TR) -> Net-(U2-THR)
- U2 pad 6: Net-(U2-DIS) -> Net-(U2-THR)
- U2 pad 7: Net-(U2-DIS) -> Net-(F2-P)
Routing:
- net GND: track 122.8 -> 92.4 mm
- net Net-(F2-P): track 0.00 -> 18.6 mm
- net Net-(U2-DIS): track 16.2 -> 0.00 mm
- net Net-(U2-TR): track 16.2 -> 0.00 mm
- net Net-(U2-THR): track 0.00 -> 13.9 mm
- net Net-(J21-P): track 10.5 -> 0.00 mm
- net Net-(C4-Pad1): track 0.00 -> 7.46 mm
- net Net-(G3-P): track 8.19 -> 13.0 mm
- net Net-(U2-R): track 53.7 -> 49.6 mm
