File: Analog_Sandbox_PCB/Analog_Sandbox_PCB.kicad_pcb (KiCad board)
At the start: 2 copper layers, 203.2 x 101.6 mm, 100 parts, among them K1 PAD, K2 PAD, K3 PAD, M1 PAD, M2 PAD, M3 PAD, Q1 2N3904, U1 Current Source, U2 NE555P

Commit message: final changes addded
Parts:
- added M4: PAD, TestPoint:TestPoint_Loop_D2.50mm_Drill1.85mm, F.Cu at (174.2, 68.0)
- added M5: PAD, TestPoint:TestPoint_Loop_D2.50mm_Drill1.85mm, F.Cu at (174.5, 83.5)
- added R22: 1000, Resistor_SMD:R_1206_3216Metric, F.Cu at (174.5, 77.8)
- moved R20 8.25 mm to (166.0, 94.5)
- moved U1 7.44 mm to (174.5, 88.8)
Connections:
- R14 pad 2: Net-(U1-V+) -> Net-(M4-P)
- R15 pad 1: Net-(U1-V+) -> Net-(M4-P)
- U1 pad 1: Net-(U1-V+) -> Net-(M5-P)
Routing:
- net GND: track 92.4 -> 72.7 mm
- net Net-(U1-V+): track 15.3 -> 0.00 mm
- net Net-(M4-P): track 0.00 -> 14.6 mm
- net Net-(M5-P): track 0.00 -> 9.54 mm
- net Net-(U1-R): track 8.92 -> 10.3 mm
Other:
- board text added: "BJT Transistor"
- board text removed: "Dependent Voltage Source"

Commit message: arch logo added
Parts:
- added G***: LOGO, LOGO, F.Cu at (63.5, 141.0)
Other:
- board text added: "Be UGA's Finest"
- board text added: "Fundamental Trainer for Circuits"
- board text removed: "Circuit Fundamental Trainer"
