File: Analog_Sandbox_PCB/Analog_Sandbox_PCB.kicad_sch (KiCad schematic)
At the start: 95 parts, among them J1 PAD, J10 PAD, J13 PAD, J14 PAD, J15 PAD, J16 PAD, J19 PAD, J2 PAD, J20 PAD, J23 PAD, J25 PAD, J27 PAD, J28 PAD, J29 PAD, J3 PAD, J31 PAD, J32 PAD, J33 PAD, J34 PAD, J35 PAD, J36 PAD, J37 PAD, J38 PAD, J39 PAD, J41 PAD, J42 PAD, J44 PAD, J45 PAD, J46 PAD, U1 555_DIP, U2 LM358_SOIC

Commit message: started schematic layout
Parts:
- removed C1: CCHIP-0402(1005-METRIC), Analog_Sandbox_PCB:CAPC1005X60, symbol Analog_Sandbox_PCB-eagle-import:CCHIP-0402(1005-METRIC)
- removed C2, C3, C4, C5, C6: CCHIP-0402(1005-METRIC), Analog_Sandbox_PCB:CAPC1005X60, symbol Analog_Sandbox_PCB-eagle-import:Tutorial - Fusion 360_16997205_CCHIP-0402(1005-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
- removed D1, D10, D2, D3, D4, D5, D6, D8, D9: CHIP-FLAT-Y_0603-0.35MM, Analog_Sandbox_PCB:LEDC1608X35N_FLAT-Y, symbol Analog_Sandbox_PCB-eagle-import:CHIP-FLAT-Y_0603-0.35MM
- removed D11, D12: DIODEDO-213AA(SOD-80), Analog_Sandbox_PCB:DIOMELF3516, symbol Analog_Sandbox_PCB-eagle-import:DIODEDO-213AA(SOD-80)
- removed D7: LED_CHIPRED-1608, Analog_Sandbox_PCB:LEDC1608X39N_R, symbol Analog_Sandbox_PCB-eagle-import:LED_CHIPRED-1608
- removed J1, J10, J13, J14, J15, J16, J19, J2, J20, J23, J25, J27, J28, J29, J3, J31, J32, J33, J34, J35, J36, J37, J38, J39, J41, J42, J44, J45, J46: PAD, Analog_Sandbox_PCB:2.54_1.0, symbol Analog_Sandbox_PCB-eagle-import:PAD
- removed R1, R10, R11, R3: 1000, Analog_Sandbox_PCB:RESC1005X40, symbol Analog_Sandbox_PCB-eagle-import:R-USCHIP-0402(1005-METRIC)
- removed R12, R13, R18, R19, R22, R23, R24, R25, R27, R28, R30, R31, R32, R34, R35: R-USCHIP-0402(1005-METRIC), Analog_Sandbox_PCB:RESC1005X40, symbol Analog_Sandbox_PCB-eagle-import:R-USCHIP-0402(1005-METRIC)
- removed R2, R4, R8: 2000, Analog_Sandbox_PCB:RESC1005X40, symbol Analog_Sandbox_PCB-eagle-import:R-USCHIP-0402(1005-METRIC)
- removed R26, R37, R5, R6: 560, Analog_Sandbox_PCB:RESC1005X40, symbol Analog_Sandbox_PCB-eagle-import:R-USCHIP-0402(1005-METRIC)
- removed R7: 3000, Analog_Sandbox_PCB:RESC1005X40, symbol Analog_Sandbox_PCB-eagle-import:R-USCHIP-0402(1005-METRIC)
- removed R9: 6000, Analog_Sandbox_PCB:RESC1005X40, symbol Analog_Sandbox_PCB-eagle-import:R-USCHIP-0402(1005-METRIC)
- removed S10, S11, S12, S13, S14, S15, S16, S17, S18, S19, S3, S4, S5, S6, S7, S8, S9: DS01E, Analog_Sandbox_PCB:DS-01, symbol Analog_Sandbox_PCB-eagle-import:DS01E
- removed U$1: BATTERYGENERIC, Analog_Sandbox_PCB:BATTERY-GENERIC, symbol Analog_Sandbox_PCB-eagle-import:BATTERYGENERIC
- removed U1: 555_DIP, Analog_Sandbox_PCB:DIP826W53P254L959H508Q8B, symbol Analog_Sandbox_PCB-eagle-import:555_DIP
- removed U2: LM358_SOIC, Analog_Sandbox_PCB:SOIC127P600X175-8N, symbol Analog_Sandbox_PCB-eagle-import:LM358_SOIC
- added B1: ~, Battery:BatteryHolder_MYOUNG_BS-07-A1BJ001_CR2032, symbol Analog_Sandbox_PCB-eagle-import:BATTERYGENERIC
- added C2, C3: C, Capacitor_SMD:C_0805_2012Metric_Pad1.18x1.45mm_HandSolder, symbol Device:C
- added R1, R2: R, Resistor_SMD:R_2010_5025Metric_Pad1.40x2.65mm_HandSolder, symbol Device:R
- added VR1: <OUTPUT VOLTAGE>, Analog_Sandbox_PCB:TO254P1054X470X1955-3, symbol Analog_Sandbox_PCB-eagle-import:LM317T
Connections:
- new net: R1.2, R2.2, VR1.1 (ADJ)
- new net GND: B1.-, C2.2, C3.2, R2.1
- new net V_Reg_Out: C2.1, R1.1, VR1.2 (VOUT)
- new net Vin: B1.+, C3.1, VR1.3 (VIN)
Other:
- added sheet DC Time Constant (dc_time_constant.kicad_sch)
- added sheet Dependent Voltage Source (dependent_voltage_source.kicad_sch)
- added sheet Mixed DC (mixed_dc.kicad_sch)
- added sheet Series and Parallel (series_and_parallel.kicad_sch)
- added sheet Thevenin (thevenin.kicad_sch)
- added sheet Through and Across (through_and_across.kicad_sch)
- added sheet Voltage Divider (voltage_divider.kicad_sch)

Commit message: All Circuits Added, Layout Almost done
Parts:
- VR1: footprint Analog_Sandbox_PCB:TO254P1054X470X1955-3 -> TRIM_3362P-1-102LF_vf.A5S3VpQGRRqLSuxbPYtLvA
Other:
- sheet DC Time Constant renamed RC Time Constant
Changed lines of the file:
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@@
 			)
 		)
-		(property "Footprint" "Analog_Sandbox_PCB:TO254P1054X470X1955-3"
+		(property "Footprint" "TRIM_3362P-1-102LF_vf.A5S3VpQGRRqLSuxbPYtLvA"
 			(at 69.85 80.01 0)
 			(effects
@@
 			(color 0 0 0 0.0000)
 		)
-		(property "Sheetname" "DC Time Constant"
+		(property "Sheetname" "RC Time Constant"
 			(at 157.48 117.3984 0)
 			(effects

Commit message: fin
Parts:
- removed B1: ~, Battery:BatteryHolder_MYOUNG_BS-07-A1BJ001_CR2032, symbol Analog_Sandbox_PCB-eagle-import:BATTERYGENERIC
- removed C2, C3: C, Capacitor_SMD:C_0805_2012Metric_Pad1.18x1.45mm_HandSolder, symbol Device:C
- removed R1, R2: R, Resistor_SMD:R_2010_5025Metric_Pad1.40x2.65mm_HandSolder, symbol Device:R
- removed VR1: <OUTPUT VOLTAGE>, TRIM_3362P-1-102LF_vf.A5S3VpQGRRqLSuxbPYtLvA, symbol Analog_Sandbox_PCB-eagle-import:LM317T
- added BT1, BT2: Battery_Cell, Battery:BatteryHolder_Keystone_1060_1x2032, symbol Device:Battery_Cell
Connections:
- net GND: now also BT1.2 (-)
- net V_Reg_Out: now also BT2.1 (+)
- new net: BT1.1 (+), BT2.2 (-)
