File: Analog_Sandbox_PCB/dc_time_constant.kicad_sch (KiCad schematic)
At the start: 1 part

Commit message: All Circuits Added, Layout Almost done
Parts:
- added C1: 0.01u, symbol Device:C
- added C4: 47u, symbol Device:C
- added D9: LED, Diode_SMD:D_1206_3216Metric, symbol Device:LED
- added R22, R23: 10k, Resistor_SMD:R_2010_5025Metric_Pad1.40x2.65mm_HandSolder, symbol Device:R
- added R24: 220, Resistor_SMD:R_2010_5025Metric_Pad1.40x2.65mm_HandSolder, symbol Device:R
- added S15: SWITCH, Button_Switch_THT:SW_DIP_SPSTx01_Slide_9.78x4.72mm_W7.62mm_P2.54mm, symbol Analog_Sandbox_PCB-eagle-import:DS01E
- added U2: NE555P, Package_DIP:DIP-8_W7.62mm, symbol Timer:NE555P
- added VR7: 100k, Analog_Sandbox_PCB:TRIM_3362P-1-102LF, symbol Analog_Sandbox_PCB-eagle-import:3362P-1-102LF
- S10: value ~ -> SWITCH; footprint Analog_Sandbox_PCB:DS-01 -> Button_Switch_THT:SW_DIP_SPSTx01_Slide_9.78x4.72mm_W7.62mm_P2.54mm
Connections:
- net V_Reg_In: now also S15.1; no longer S10.1
- net at S10.2: now also R22.2, U2.2 (TR)
- new net: R23.2, S10.1, S15.2, U2.4 (R), U2.8 (VCC)
- new net: C4.1, U2.6 (THR), U2.7 (DIS), VR7.2 (WIPER)
- new net: R23.1, VR7.1 (CCW)
- new net: C1.1, U2.5 (CV)
- new net: D9.2 (A), R24.2
- new net: R24.1, U2.3 (Q)
- new net GND: C1.2, C4.2, D9.1 (K), R22.1, U2.1 (GND), VR7.3 (CW)

Commit message: fin
Parts:
- removed VR7: 100k, Analog_Sandbox_PCB:TRIM_3362P-1-102LF, symbol Analog_Sandbox_PCB-eagle-import:3362P-1-102LF
- added D11: LED, Diode_SMD:D_1206_3216Metric, symbol Device:LED
- added J21, Q2: PAD, TestPoint:TestPoint_Loop_D2.50mm_Drill1.85mm, symbol Analog_Sandbox_PCB-eagle-import:PAD
- added R2: 560, Resistor_SMD:R_1206_3216Metric, symbol Device:R
- added R35: 3362P-1-103LF, Sandbox:POT_3362P, symbol 3362p:3362P-1-103LF
- C1, C4: footprint (none) -> Capacitor_SMD:C_1206_3216Metric
- R22, R23, R24: footprint Resistor_SMD:R_2010_5025Metric_Pad1.40x2.65mm_HandSolder -> Resistor_SMD:R_1206_3216Metric
Connections:
- net GND: now also D11.1 (K), R35.1
- net at R23.2, S10.1, S15.2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: now also R2.1
- net at C4.1, U2.6 (THR), U2.7 (DIS): now also R35.2
- net at R23.1: now also J21.1 (P), R35.3
- net at R24.1, U2.3 (Q): now also Q2.1 (P)
- new net: D11.2 (A), R2.2

Commit message: made changes from morning of 4/13
Parts:
- removed R22: 10k, Resistor_SMD:R_1206_3216Metric, symbol Device:R
- removed S10: SWITCH, Button_Switch_THT:SW_DIP_SPSTx01_Slide_9.78x4.72mm_W7.62mm_P2.54mm, symbol Analog_Sandbox_PCB-eagle-import:DS01E
- renumbered Q2 to F1, J21 to F2
Connections:
- net GND: no longer R35.1
- net at F2.1 (P), R23.1, R35.3: now also U2.7 (DIS)
- net at R35.2, U2.6 (THR): now also U2.2 (TR); no longer C4.1, U2.7 (DIS)
- new net: C4.1, R35.1
Other:
- moved on the sheet: C4, R35
