File: Analog_Sandbox_PCB/dependent_voltage_source.kicad_sch (KiCad schematic)
At the start: 0 parts

Commit message: All Circuits Added, Layout Almost done
Parts:
- added J18, J19: PAD, Analog_Sandbox_PCB:2.54_1.0, symbol Analog_Sandbox_PCB-eagle-import:PAD
- added Q1: 2N3904, Package_TO_SOT_THT:TO-92_Inline, symbol Transistor_BJT:2N3904
- added R28: 4.7k, Resistor_SMD:R_2010_5025Metric_Pad1.40x2.65mm_HandSolder, symbol Device:R
- added R29: 1k, Resistor_SMD:R_2010_5025Metric_Pad1.40x2.65mm_HandSolder, symbol Device:R
- added S19: SWITCH, Button_Switch_THT:SW_DIP_SPSTx01_Slide_9.78x4.72mm_W7.62mm_P2.54mm, symbol Analog_Sandbox_PCB-eagle-import:DS01E
- added VR9: 10k, Analog_Sandbox_PCB:TRIM_3362P-1-102LF, symbol Analog_Sandbox_PCB-eagle-import:3362P-1-102LF
Connections:
- net V_Reg_In: now also S19.1
- new net: Q1.3 (C), S19.2, VR9.3 (CW)
- new net: J19.1 (P), R28.2, VR9.2 (WIPER)
- new net: J18.1 (P), Q1.1 (E), R29.1
- new net: Q1.2 (B), R28.1
- new net GND: R29.2, VR9.1 (CCW)

Commit message: fin
Parts:
- removed J19: PAD, Analog_Sandbox_PCB:2.54_1.0, symbol Analog_Sandbox_PCB-eagle-import:PAD
- removed VR9: 10k, Analog_Sandbox_PCB:TRIM_3362P-1-102LF, symbol Analog_Sandbox_PCB-eagle-import:3362P-1-102LF
- added Base1: PAD, TestPoint:TestPoint_Loop_D2.50mm_Drill1.85mm, symbol Analog_Sandbox_PCB-eagle-import:PAD
- added D12: LED, Diode_SMD:D_1206_3216Metric, symbol Device:LED
- added R36: 3362P-1-103LF, Sandbox:POT_3362P, symbol 3362p:3362P-1-103LF
- added R38: 560, Resistor_SMD:R_1206_3216Metric, symbol Device:R
- Emitter1: renamed from J18; footprint Analog_Sandbox_PCB:2.54_1.0 -> TestPoint:TestPoint_Loop_D2.50mm_Drill1.85mm
- Q1: footprint Package_TO_SOT_THT:TO-92_Inline -> Connector_PinHeader_2.54mm:PinHeader_1x03_P2.54mm_Vertical
- R28, R29: footprint Resistor_SMD:R_2010_5025Metric_Pad1.40x2.65mm_HandSolder -> Resistor_SMD:R_1206_3216Metric
Connections:
- net GND: now also D12.1 (K), R36.3
- net at Q1.3 (C), S19.2: now also R36.1, R38.1
- net at R28.2: now also Base1.1 (P), R36.2
- new net: D12.2 (A), R38.2

Commit message: made changes from morning of 4/13
Parts:
- added G1, G3: PAD, TestPoint:TestPoint_Loop_D2.50mm_Drill1.85mm, symbol Analog_Sandbox_PCB-eagle-import:PAD
- renumbered Base1 to G2, Emitter1 to G4
Connections:
- net at Q1.3 (C), R36.1, R38.1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: now also G1.1 (P)
- net at Q1.2 (B), R28.1: now also G3.1 (P)
Changed lines of the file:
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@@
+	)
+	(junction
+		(at 72.39 44.45)
+		(diameter 0)
+		(color 0 0 0 0)
+	)
+	(junction
+		(at 83.82 33.02)
+		(diameter 0)
+		(color 0 0 0 0)
 	)
 	(junction
@@
 	(wire
 		(pts
+			(xy 72.39 40.64) (xy 72.39 44.45)
+		)
+		(stroke
+			(width 0)
+			(type default)
+		)
+	)
+	(wire
+		(pts
 			(xy 83.82 49.53) (xy 83.82 50.8)
 		)
@@
 	(wire
 		(pts
-			(xy 71.12 44.45) (xy 76.2 44.45)
+			(xy 71.12 44.45) (xy 72.39 44.45)
 		)
 		(stroke
@@
 		(pts
 			(xy 45.72 33.02) (xy 48.26 33.02)
+		)
+		(stroke
+			(width 0)
+			(type default)
+		)
+	)
+	(wire
+		(pts
+			(xy 72.39 44.45) (xy 76.2 44.45)
 		)
 		(stroke
@@
 	(symbol
 		(lib_id "Analog_Sandbox_PCB-eagle-import:PAD")
+		(at 72.39 38.1 270)
+		(unit 1)
+		(exclude_from_sim no)
+		(in_bom yes)
+		(on_board yes)
+		(dnp no)
+		(fields_autoplaced yes)
+		(property "Reference" "G3"
+			(at 74.93 36.195 90)
+			(effects
+				(font
+					(size 1.778 1.5113)
+				)
+				(justify left)
+			)
+		)
+		(property "Value" "PAD"
+			(at 74.93 40.005 90)
+			(effects
+				(font
+					(size 1.778 1.5113)
+				)
+				(justify left)
+			)
+		)
+		(property "Footprint" "TestPoint:TestPoint_Loop_D2.50mm_Drill1.85mm"
+			(at 72.39 38.1 0)
+			(effects
+				(font
+					(size 1.27 1.27)
+				)
+				(hide yes)
+			)
+		)
+		(property "Datasheet" ""
+			(at 72.39 38.1 0)
+			(effects
+				(font
+					(size 1.27 1.27)
+				)
+				(hide yes)
+			)
+		)
+		(property "Description" ""
+			(at 72.39 38.1 0)
+			(effects
+				(font
+					(size 1.27 1.27)
+				)
+				(hide yes)
+			)
+		)
+		(pin "1"
+		)
+		(instances
+			(project "Analog_Sandbox_PCB"
+				(path "/ac750111-a1db-4b3c-a106-e1424e47aebb/fe66ce79-8177-44fa-a561-9cdc131a7718"
+					(reference "G3")
+					(unit 1)
+				)
+			)
+		)
+	)
+	(symbol
+		(lib_id "Analog_Sandbox_PCB-eagle-import:PAD")
 		(at 58.42 38.1 270)
 		(unit 1)
@@
 		(on_board yes)
 		(dnp no)
-		(fields_autoplaced yes)
-		(property "Reference" "Base1"
-			(at 60.96 36.195 90)
+		(property "Reference" "G2"
+			(at 61.214 36.068 90)
 			(effects
 				(font
@@
 			(project "Analog_Sandbox_PCB"
 				(path "/ac750111-a1db-4b3c-a106-e1424e47aebb/fe66ce79-8177-44fa-a561-9cdc131a7718"
-					(reference "Base1")
+					(reference "G2")
 					(unit 1)
 				)
@@
 	)
 	(symbol
+		(lib_id "Analog_Sandbox_PCB-eagle-import:PAD")
+		(at 86.36 33.02 180)
+		(unit 1)
+		(exclude_from_sim no)
+		(in_bom yes)
+		(on_board yes)
+		(dnp no)
+		(fields_autoplaced yes)
+		(property "Reference" "G1"
+			(at 88.9 31.115 0)
+			(effects
+				(font
+					(size 1.778 1.5113)
+				)
+				(justify right)
+			)
+		)
+		(property "Value" "PAD"
+			(at 88.9 34.925 0)
+			(effects
+				(font
+					(size 1.778 1.5113)
+				)
+				(justify right)
+			)
+		)
+		(property "Footprint" "TestPoint:TestPoint_Loop_D2.50mm_Drill1.85mm"
+			(at 86.36 33.02 0)
+			(effects
+				(font
+					(size 1.27 1.27)
+				)
+				(hide yes)
+			)
+		)
+		(property "Datasheet" ""
+			(at 86.36 33.02 0)
+			(effects
+				(font
+					(size 1.27 1.27)
+				)
+				(hide yes)
+			)
+		)
+		(property "Description" ""
+			(at 86.36 33.02 0)
+			(effects
+				(font
+					(size 1.27 1.27)
+				)
+				(hide yes)
+			)
+		)
+		(pin "1"
+		)
+		(instances
+			(project "Analog_Sandbox_PCB"
+				(path "/ac750111-a1db-4b3c-a106-e1424e47aebb/fe66ce79-8177-44fa-a561-9cdc131a7718"
+					(reference "G1")
+					(unit 1)
+				)
+			)
+		)
+	)
+	(symbol
 		(lib_id "3362p:3362P-1-103LF")
 		(at 50.8 34.29 270)
@@
 		(dnp no)
 		(fields_autoplaced yes)
-		(property "Reference" "Emitter1"
+		(property "Reference" "G4"
 			(at 93.98 48.895 0)
 			(effects
@@
 			(project "Analog_Sandbox_PCB"
 				(path "/ac750111-a1db-4b3c-a106-e1424e47aebb/fe66ce79-8177-44fa-a561-9cdc131a7718"
-					(reference "Emitter1")
-					(unit 1)
-				)
+					(reference "G4")
+					(unit 1)
+				)
