File: Analog_Sandbox_PCB/series_and_parallel.kicad_sch (KiCad schematic)
At the start: 19 parts, among them J12 PAD, J13 PAD, J14 PAD, J15 PAD, J16 PAD

Commit message: All Circuits Added, Layout Almost done
Parts:
- removed D5, D6, D7, D8: ~, Diode_SMD:D_2010_5025Metric_Pad1.52x2.65mm_HandSolder, symbol Analog_Sandbox_PCB-eagle-import:CHIP-FLAT-Y_0603-0.35MM
- added D5, D6, D7, D8: LED, Diode_SMD:D_1206_3216Metric, symbol Device:LED
- added R21: 100, Resistor_SMD:R_2010_5025Metric_Pad1.40x2.65mm_HandSolder, symbol Device:R
- added S11, S12, S13, S14: SWITCH, Button_Switch_THT:SW_DIP_SPSTx01_Slide_9.78x4.72mm_W7.62mm_P2.54mm, symbol Analog_Sandbox_PCB-eagle-import:DS01E
- J14, J16: footprint Analog_Sandbox_PCB:2.54_1.0 -> 2.54_1.0_16378166
- R16, R17, R18, R19: value R -> 100
- S8, S9: footprint Analog_Sandbox_PCB:DS-01 -> Button_Switch_THT:SW_DIP_SPSTx01_Slide_9.78x4.72mm_W7.62mm_P2.54mm
- VR3, VR5, VR6: footprint Analog_Sandbox_PCB:TRIM_3362P-1-102LF -> TRIM_3362P-1-102LF_vf.A5S3VpQGRRqLSuxbPYtLvA
Connections:
- net GND: now also S9.1; no longer S9.2
- net at VR4.1 (CCW): no longer R17.2
- net at VR4.2 (WIPER): now also D6.2 (A)
- net at VR4.3 (CW): now also R17.2
- net at J12.1 (P), R16.1: now also R21.1, S11.1; no longer S8.2
- net at J15.1 (P), R19.2: now also D6.1 (K), S12.2, S13.1
- net at J14.1 (P), R17.1, R18.2: now also D5.1 (K), S11.2, S12.1, S14.1
- net at J13.1 (P): now also J16.1 (P), S9.2, D7.1 (K), D8.1 (K), S13.2, S14.2
- net at VR5.2 (WIPER): now also D7.2 (A)
- net at VR3.3 (CW): now also R16.2
- net at VR3.1 (CCW): no longer R16.2
- net at VR3.2 (WIPER): now also D5.2 (A)
- net at VR6.2 (WIPER): now also D8.2 (A)
- new net: R21.2, S8.2
Other:
- moved on the sheet: J16, VR3, VR5, VR6

Commit message: fin
Parts:
- removed J16: PAD, 2.54_1.0_16378166, symbol Analog_Sandbox_PCB-eagle-import:PAD
- removed VR3, VR5, VR6: ~, TRIM_3362P-1-102LF_vf.A5S3VpQGRRqLSuxbPYtLvA, symbol Analog_Sandbox_PCB-eagle-import:3362P-1-102LF
- removed VR4: ~, Analog_Sandbox_PCB:TRIM_3362P-1-102LF, symbol Analog_Sandbox_PCB-eagle-import:3362P-1-102LF
- added D10: LED, Diode_SMD:D_1206_3216Metric, symbol Device:LED
- added R1: 560, Resistor_SMD:R_1206_3216Metric, symbol Device:R
- added R30, R32, R33, R34: 3362P-1-103LF, Sandbox:POT_3362P, symbol 3362p:3362P-1-103LF
- J12, J13, J15: footprint Analog_Sandbox_PCB:2.54_1.0 -> TestPoint:TestPoint_Loop_D2.50mm_Drill1.85mm
- J14: footprint 2.54_1.0_16378166 -> TestPoint:TestPoint_Loop_D2.50mm_Drill1.85mm
- R16, R17, R18, R19, R21: footprint Resistor_SMD:R_2010_5025Metric_Pad1.40x2.65mm_HandSolder -> Resistor_SMD:R_1206_3216Metric
Connections:
- net GND: now also D10.1 (K), R30.3, R32.3, R33.3, R34.3
- net at R21.2, S8.2: now also R1.1
- net at R18.1: now also R33.1
- net at D6.2 (A): now also R30.2
- net at R17.2: now also R30.1
- net at D7.2 (A): now also R33.2
- net at D8.2 (A): now also R34.2
- net at D5.2 (A): now also R32.2
- net at R16.2: now also R32.1
- net at R19.1: now also R34.1
- new net: D10.2 (A), R1.2

Commit message: made changes from morning of 4/13
Parts:
- renumbered J12 to E1, J14 to E2, J15 to E3, J13 to E4
Changed lines of the file:
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@@
 		(dnp no)
 		(fields_autoplaced yes)
-		(property "Reference" "J14"
+		(property "Reference" "E2"
 			(at 104.14 40.005 90)
 			(effects
@@
 			(project "Analog_Sandbox_PCB"
 				(path "/ac750111-a1db-4b3c-a106-e1424e47aebb/ea0b2902-1294-499d-a00b-a55787386bf7"
-					(reference "J14")
+					(reference "E2")
 					(unit 1)
 				)
@@
 		(dnp no)
 		(fields_autoplaced yes)
-		(property "Reference" "J12"
+		(property "Reference" "E1"
 			(at 41.91 36.83 0)
 			(effects
@@
 			(project "Analog_Sandbox_PCB"
 				(path "/ac750111-a1db-4b3c-a106-e1424e47aebb/ea0b2902-1294-499d-a00b-a55787386bf7"
-					(reference "J12")
+					(reference "E1")
 					(unit 1)
 				)
@@
 		(dnp no)
 		(fields_autoplaced yes)
-		(property "Reference" "J13"
+		(property "Reference" "E4"
 			(at 166.37 98.425 90)
 			(effects
@@
 			(project "Analog_Sandbox_PCB"
 				(path "/ac750111-a1db-4b3c-a106-e1424e47aebb/ea0b2902-1294-499d-a00b-a55787386bf7"
-					(reference "J13")
+					(reference "E4")
 					(unit 1)
 				)
@@
 		(dnp no)
 		(fields_autoplaced yes)
-		(property "Reference" "J15"
+		(property "Reference" "E3"
 			(at 166.37 38.735 90)
 			(effects
@@
 			(project "Analog_Sandbox_PCB"
 				(path "/ac750111-a1db-4b3c-a106-e1424e47aebb/ea0b2902-1294-499d-a00b-a55787386bf7"
-					(reference "J15")
-					(unit 1)
-				)
+					(reference "E3")
+					(unit 1)
+				)
