File: Analog_Sandbox_PCB/voltage_divider.kicad_sch (KiCad schematic)
At the start: 14 parts, among them J4 PAD, J5 PAD, J6 PAD, J7 PAD

Commit message: slight update
Parts:
- J4, J5, J6, J7: footprint Analog_Sandbox_PCB:2.54_1.0 -> TestPoint:TestPoint_Pad_2.5x2.5mm
- R12, R7, R8: footprint Resistor_SMD:R_2010_5025Metric_Pad1.40x2.65mm_HandSolder -> Resistor_SMD:R_1206_3216Metric
- S2, S3: footprint Analog_Sandbox_PCB:DS-01 -> Button_Switch_THT:SW_DIP_SPSTx01_Slide_9.78x4.72mm_W7.62mm_P2.54mm
Connections:
- net GND: now also J4.1 (P); no longer J7.1 (P)
- net at S2.1: now also J6.1 (P), R7.2, R8.1
- net at S3.1: now also J5.1 (P), R8.2, R9.1
- net at R12.1, S4.2: now also J7.1 (P), R7.1

Commit message: Config LM134
Parts:
- S4: footprint Analog_Sandbox_PCB:DS-01 -> Button_Switch_THT:SW_DIP_SPSTx01_Slide_9.78x4.72mm_W7.62mm_P2.54mm

Commit message: All Circuits Added, Layout Almost done
Parts:
- removed D3: LED, Diode_SMD:D_2010_5025Metric_Pad1.52x2.65mm_HandSolder, symbol Analog_Sandbox_PCB-eagle-import:CHIP-FLAT-Y_0603-0.35MM
- added D3: LED, Diode_SMD:D_1206_3216Metric, symbol Device:LED
Connections:
- net GND: now also D3.1 (K)
- net at R12.2: now also D3.2 (A)
Changed lines of the file:
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@@
+	)
+	(junction
+		(at 96.52 26.67)
+		(diameter 0)
+		(color 0 0 0 0)
 	)
 	(junction
@@
 	)
 	(junction
+		(at 104.14 26.67)
+		(diameter 0)
+		(color 0 0 0 0)
+	)
+	(junction
 		(at 80.01 26.67)
 		(diameter 0)
@@
 	(wire
 		(pts
-			(xy 105.41 26.67) (xy 102.87 26.67)
+			(xy 105.41 26.67) (xy 104.14 26.67)
 		)
 		(stroke
@@
 	(wire
 		(pts
+			(xy 96.52 26.67) (xy 97.79 26.67)
+		)
+		(stroke
+			(width 0)
+			(type default)
+		)
+	)
+	(wire
+		(pts
 			(xy 82.55 93.98) (xy 96.52 93.98)
 		)
@@
 	(wire
 		(pts
-			(xy 93.98 26.67) (xy 97.79 26.67)
+			(xy 93.98 26.67) (xy 96.52 26.67)
 		)
 		(stroke
@@
 		(pts
 			(xy 96.52 49.53) (xy 96.52 44.45)
+		)
+		(stroke
+			(width 0)
+			(type default)
+		)
+	)
+	(wire
+		(pts
+			(xy 104.14 26.67) (xy 102.87 26.67)
 		)
 		(stroke
@@
 			)
 			(justify right)
-		)
-	)
-	(symbol
-		(lib_id "Analog_Sandbox_PCB-eagle-import:CHIP-FLAT-Y_0603-0.35MM")
-		(at 100.33 26.67 0)
-		(unit 1)
-		(exclude_from_sim no)
-		(in_bom yes)
-		(on_board yes)
-		(dnp no)
-		(fields_autoplaced yes)
-		(property "Reference" "D3"
-			(at 100.33 17.78 0)
-			(effects
-				(font
-					(size 1.778 1.5113)
-				)
-			)
-		)
-		(property "Value" "LED"
-			(at 100.33 21.59 0)
-			(effects
-				(font
-					(size 1.778 1.5113)
-				)
-			)
-		)
-		(property "Footprint" "Diode_SMD:D_2010_5025Metric_Pad1.52x2.65mm_HandSolder"
-			(at 100.33 26.67 0)
-			(effects
-				(font
-					(size 1.27 1.27)
-				)
-				(hide yes)
-			)
-		)
-		(property "Datasheet" ""
-			(at 100.33 26.67 0)
-			(effects
-				(font
-					(size 1.27 1.27)
-				)
-				(hide yes)
-			)
-		)
-		(property "Description" "Yellow LED - Generic"
-			(at 100.33 26.67 0)
-			(effects
-				(font
-					(size 1.27 1.27)
-				)
-				(hide yes)
-			)
-		)
-		(pin "A"
-		)
-		(pin "C"
-		)
-		(instances
-			(project "Analog_Sandbox_PCB"
-				(path "/ac750111-a1db-4b3c-a106-e1424e47aebb/9c122918-2265-473b-8c84-35fbd0d69d38"
-					(reference "D3")
-					(unit 1)
-				)
-			)
 		)
 	)
@@
 					(unit 1)
 				)
+			)
+		)
+	)
+	(symbol
+		(lib_id "Device:LED")
+		(at 100.33 26.67 180)
+		(unit 1)
+		(exclude_from_sim no)
+		(in_bom yes)
+		(on_board yes)
+		(dnp no)
+		(fields_autoplaced yes)
+		(property "Reference" "D3"
+			(at 101.9175 19.05 0)
+			(effects
+				(font
+					(size 1.27 1.27)
+				)
+			)
+		)
+		(property "Value" "LED"
+			(at 101.9175 21.59 0)
+			(effects
+				(font
+					(size 1.27 1.27)
+				)
+			)
+		)
+		(property "Footprint" "Diode_SMD:D_1206_3216Metric"
+			(at 100.33 26.67 0)
+			(effects
+				(font
+					(size 1.27 1.27)
+				)
+				(hide yes)
+			)
+		)
+		(property "Datasheet" "~"
+			(at 100.33 26.67 0)
+			(effects
+				(font
+					(size 1.27 1.27)
+				)
+				(hide yes)
+			)
+		)
+		(property "Description" "Light emitting diode"
+			(at 100.33 26.67 0)
+			(effects
+				(font
+					(size 1.27 1.27)
+				)
+				(hide yes)
+			)
+		)
+		(property "Sim.Pins" "1=K 2=A"
+			(at 100.33 26.67 0)
+			(effects
+				(font
+					(size 1.27 1.27)
+				)
+				(hide yes)
+			)
+		)
+		(pin "1"
+		)
+		(pin "2"
+		)
+		(instances
+			(project "Analog_Sandbox_PCB"
+				(path "/ac750111-a1db-4b3c-a106-e1424e47aebb/9c122918-2265-473b-8c84-35fbd0d69d38"
+					(reference "D3")
+					(unit 1)
+				)

Commit message: fin
Parts:
- J4, J5, J6, J7: footprint TestPoint:TestPoint_Pad_2.5x2.5mm -> TestPoint:TestPoint_Loop_D2.50mm_Drill1.85mm
- R10, R11, R9: footprint Resistor_SMD:R_2010_5025Metric_Pad1.40x2.65mm_HandSolder -> Resistor_SMD:R_1206_3216Metric

Commit message: made changes from morning of 4/13
Parts:
- renumbered J7 to B1, J6 to B2, J5 to B3, J4 to B4
Changed lines of the file:
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@@
 		(dnp no)
 		(fields_autoplaced yes)
-		(property "Reference" "J7"
+		(property "Reference" "B1"
 			(at 82.55 45.085 90)
 			(effects
@@
 			(project "Analog_Sandbox_PCB"
 				(path "/ac750111-a1db-4b3c-a106-e1424e47aebb/9c122918-2265-473b-8c84-35fbd0d69d38"
-					(reference "J7")
+					(reference "B1")
 					(unit 1)
 				)
@@
 		(dnp no)
 		(fields_autoplaced yes)
-		(property "Reference" "J6"
+		(property "Reference" "B2"
 			(at 93.98 52.07 0)
 			(effects
@@
 			(project "Analog_Sandbox_PCB"
 				(path "/ac750111-a1db-4b3c-a106-e1424e47aebb/9c122918-2265-473b-8c84-35fbd0d69d38"
-					(reference "J6")
+					(reference "B2")
 					(unit 1)
 				)
@@
 		(dnp no)
 		(fields_autoplaced yes)
-		(property "Reference" "J4"
+		(property "Reference" "B4"
 			(at 99.06 94.615 90)
 			(effects
@@
 			(project "Analog_Sandbox_PCB"
 				(path "/ac750111-a1db-4b3c-a106-e1424e47aebb/9c122918-2265-473b-8c84-35fbd0d69d38"
-					(reference "J4")
+					(reference "B4")
 					(unit 1)
 				)
@@
 		(dnp no)
 		(fields_autoplaced yes)
-		(property "Reference" "J5"
+		(property "Reference" "B3"
 			(at 93.98 71.12 0)
 			(effects
@@
 			(project "Analog_Sandbox_PCB"
 				(path "/ac750111-a1db-4b3c-a106-e1424e47aebb/9c122918-2265-473b-8c84-35fbd0d69d38"
-					(reference "J5")
-					(unit 1)
-				)
+					(reference "B3")
+					(unit 1)
+				)
